File: preamp.sch (KiCad schematic (older format))
At the start: 69 parts, among them J1 AC, J2 JST_XH_3, J3 JST_XH_3, J4 JST_XH_3, J6 JST_XH_3, SW1 SW_SPST, SW2 SW_SPST, U1 L78L09_SOT89, U2 L78L05_SOT89, U3 NJM2753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

Commit message: tidied up
Connections:
- net at D1.1 (K), D3.2 (A): now also J1.1 (Pin_1); no longer J1.3 (Pin_3)
- net at D2.1 (K), D4.2 (A): now also J1.3 (Pin_3); no longer J1.1 (Pin_1)
Changed lines of the file:
@@
 EESchema Schematic File Version 4
 LIBS:preamp-cache
-EELAYER 26 0
+EELAYER 29 0
 EELAYER END
 $Descr A4 11693 8268
@@
 Wire Wire Line
 	9750 3450 9750 3475
-$Comp
-L Connector:Conn_01x03_Male J1
-U 1 1 5CD88BA8
-P 625 5650
-F 0 "J1" H 597 5582 50  0000 R CNN
-F 1 "AC" H 597 5673 50  0000 R CNN
-F 2 "Connector_JST:JST_XH_B3B-XH-A_1x03_P2.50mm_Vertical" H 625 5650 50  0001 C CNN
-F 3 "~" H 625 5650 50  0001 C CNN
-	1    625  5650
-	1    0    0    1
-$EndComp
 Wire Wire Line
 	825  5550 950  5550
@@
 Wire Wire Line
 	4650 7500 5125 7500
+$Comp
+L Connector:Conn_01x03_Male J1
+U 1 1 5CD88BA8
+P 625 5650
+F 0 "J1" H 597 5582 50  0000 R CNN
+F 1 "AC" H 597 5673 50  0000 R CNN
+F 2 "Connector_JST:JST_XH_B3B-XH-A_1x03_P2.50mm_Vertical" H 625 5650 50  0001 C CNN
+F 3 "~" H 625 5650 50  0001 C CNN
+	1    625  5650
+	1    0    0    -1
+$EndComp
 $EndSCHEMATC
