File: preamp.sch (KiCad schematic (older format))
At the start: 69 parts, among them J1 AC, J2 JST_XH_3, J3 JST_XH_3, J4 JST_XH_3, J6 JST_XH_3, SW1 SW_SPST, SW2 SW_SPST, U1 L78L09_SOT89, U2 L78L05_SOT89, U3 NJM2753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

Commit message: updated silkscreen
Parts:
- U3: symbol custom:NJM2753 -> preamp-rescue:NJM2753-custom
- U6: symbol custom:PGA2311 -> preamp-rescue:PGA2311-custom
- U8: symbol custom:OLED_128x64 -> preamp-rescue:OLED_128x64-custom
Changed lines of the file:
@@
 EESchema Schematic File Version 4
 LIBS:preamp-cache
-EELAYER 29 0
+EELAYER 26 0
 EELAYER END
 $Descr A4 11693 8268
@@
 $EndComp
 $Comp
-L custom:PGA2311 U6
+L preamp-rescue:PGA2311-custom U6
 U 1 1 5CBB4769
 P 7225 1525
@@
 $EndComp
 $Comp
-L custom:OLED_128x64 U8
+L preamp-rescue:OLED_128x64-custom U8
 U 1 1 5CD308C7
 P 11025 2900
@@
 	5000 900  5000 1325
 $Comp
-L custom:NJM2753 U3
+L preamp-rescue:NJM2753-custom U3
 U 1 1 5D00A564
 P 4025 1575

Commit message: tweaks before productioN
Parts:
- C10, C11, C12, C25, C27, C7, C8, C9: value 1u -> 4u7
- C5, C6: value 35V 1500u -> 35V 270u; footprint Capacitor_THT:CP_Radial_D10.0mm_P2.50mm -> Capacitor_SMD:CP_Elec_10x10
- D1, D2, D3, D4: value 1N4001 -> ES1JL
- R11, R12: value 100K -> 47K
Connections:
- net at C18.1, U6.16 (IN_L): now also R9.1
- net at C21.2, U6.9 (IN_R): now also R10.1
- net at C21.1, U3.14 (OUTB): no longer R10.1
- net at C18.2, U3.1 (OUTA): no longer R9.1
Other:
- moved on the sheet: C21, C22, C24, H1, H2, H3, H4, R10, R9, U4

Commit message: prototype built, tested and installed into hifi system
Parts:
- A1: symbol MCU_Module:Arduino_Nano_v3.x -> preamp-rescue:Arduino_Nano_v3.x-MCU_Module
- U6: footprint Package_SO:SOIC-16W_5.3x10.2mm_P1.27mm -> Package_SO:SOIC-16W_7.5x10.3mm_P1.27mm
Connections:
- net +5VD: now also U6.8 (~MUTE)
Other:
- note added: "1: CNT2 L CNT1 L\n2: CNT2 L CNT1 H\n3: CNT2 H CNT1 X"
- note added: "Input sockets"
- note added: "Input switching"
- note added: "MCU"
- note added: "Power"
- note added: "User input"
- note added: "Volume control"
- note added: "oops, leaving SPI pinout error for code compatibility"
- moved on the sheet: A1, C13, C14, C15, C25, C27, C28, C29, H1, J6, R11, R12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
